File: nRF24L01_mtr_driver/nRF24L01_mtr_driver.sch (KiCad schematic (older format))
At the start: 117 parts, among them J1 Micro USB, J2 I/O, J4 VBAT, J5 MTR, J6 SERVO, J7 ICSP, Q1 AO4484, Q2 AO4484, Q3 AO4484, Q4 AO4484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

Commit message: added voltage sense isolation, needs routing
Parts:
- added C44, C45, C46, C47, C48, C49: .1u, Capacitors_SMD:C_0402, symbol C
- added D8: SMA6J18AHR3G, mc-footprints:DO-214AC, symbol D_TVS
- added F1: F3542CT-ND, Resistors:1206, symbol Fuse
- added R34, R35, R36, R37: 10k, Resistors_SMD:R_0402, symbol R
- added R38: 1k, Resistors_SMD:R_0402, symbol R
- added TP1, TP3: 5V0_PWR, Measurement_Points:Measurement_Point_Square-SMD-Pad_Small, symbol TEST
- added TP2: 12V_PWR, Measurement_Points:Measurement_Point_Square-SMD-Pad_Small, symbol TEST
- added TP4: 3V3_PWR, Measurement_Points:Measurement_Point_Square-SMD-Pad_Small, symbol TEST
- added U14: ACPL-C87A, Housings_SOIC:SSO-8_6.8x5.9mm_Pitch1.27mm_Clearance8mm, symbol ACPL-C87A
- added U15: OPA237_SOT23-5, TO_SOT_Packages_SMD:SOT-23-5, symbol OPA237_SOT23-5
- R19: value 10k -> 100k
- R20: value 38k -> 12.7k
Connections:
- net 12V is gone; now on net 12V_PWR: C15.1, C25.1, D12.2 (A), D5.2 (A), R5.1, U12.1 (VDD), U5.1 (VDD)
- net 3.3V is gone; now on net 3V3_MCU: R6.1
- net 5V_MCU is gone; now on net 5V0_MCU: C35.2, C36.2, C37.2, U7.1 (VCC1), U8.1 (VCC1), U9.1 (VCC1)
- net 5V_PWR is gone; now on net 5V0_PWR: C38.2, C39.2, C40.2, U7.8 (VCC2), U8.8 (VCC2), U9.8 (VCC2)
- net 5V_mtr_driver is gone; now on net 5V0_PWR: R8.1
- net 12V_PWR: now also TP2.1
- net 3V3_MCU: now also TP4.1
- net 5V0_MCU: now also C45.1, TP3.1, U14.8 (VDD2)
- net 5V0_PWR: now also C44.1, TP1.1, U14.1 (VDD1)
- net ADC1: now also C49.1, R38.1; no longer C27.1, R19.1, R20.2
- net GNDA: now also C45.2, C46.2, C48.2, C49.2, R36.1, U14.5 (GND2), U15.2 (V-); no longer C27.2, R19.2
- net GNDPWR: now also C27.2, R20.2, C44.2, D8.1 (A1), D8.2 (A2), U14.3 (IN-), U14.4 (GND1)
- net VBAT: now also R19.1, F1.1; no longer J4.1
- net VBAT_S: no longer R20.1
- new net: F1.2, J4.1
- new net: C27.1, R19.2, R20.1, U14.2 (IN)
- new net: R34.2, U14.6 (OUT-)
- new net: R35.2, U14.7 (OUT+)
- new net: C47.1, R34.1, R37.2, U15.4 (-In)
- new net: C46.1, R35.1, R36.2, U15.3 (+In)
- new net: C47.2, R37.1, R38.2, U15.1 (Output)
- new net: C48.1, U15.5 (V+)
Other:
- note added: "3V3, 600mA\n"
- note added: "5V, 600mA"
- note added: "I/O"
- moved on the sheet: C1, C10, C11, C12, C13, C14, C15, C16, C17, C18, C19, C2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

Commit message: Changed the footprint of some 0603 cpacitors to 0402 to save space
Parts:
- C20, C30, C8: footprint Capacitors_SMD:C_0603 -> Capacitors_SMD:C_0402
- C21: footprint Capacitors_SMD:C_0805_HandSoldering -> Capacitors_SMD:C_0805
- R25: footprint Resistors_SMD:R_0603 -> Resistors_SMD:R_0402
Changed lines of the file:
@@
 F 0 "C21" H 12720 8000 50  0000 L CNN
 F 1 "4.7u" H 12720 7800 50  0000 L CNN
-F 2 "Capacitors_SMD:C_0805_HandSoldering" H 12733 7750 50  0001 C CNN
+F 2 "Capacitors_SMD:C_0805" H 12733 7750 50  0001 C CNN
 F 3 "" H 12695 7900 50  0001 C CNN
 	1    12695 7900
@@
 F 0 "C8" H 7230 12575 50  0000 L CNN
 F 1 "4.7u" H 7230 12375 50  0000 L CNN
-F 2 "Capacitors_SMD:C_0603" H 7243 12325 50  0001 C CNN
+F 2 "Capacitors_SMD:C_0402" H 7243 12325 50  0001 C CNN
 F 3 "" H 7205 12475 50  0001 C CNN
 	1    7205 12475
@@
 F 0 "C20" H 15990 16590 50  0000 L CNN
 F 1 ".1u" H 15990 16390 50  0000 L CNN
-F 2 "Capacitors_SMD:C_0603" H 16003 16340 50  0001 C CNN
+F 2 "Capacitors_SMD:C_0402" H 16003 16340 50  0001 C CNN
 F 3 "" H 15965 16490 50  0001 C CNN
 	1    15965 16490
@@
 F 0 "R25" V 8980 15000 50  0000 C CNN
 F 1 "10k" V 9030 14825 50  0000 C CNN
-F 2 "Resistors_SMD:R_0603" V 8960 14825 50  0001 C CNN
+F 2 "Resistors_SMD:R_0402" V 8960 14825 50  0001 C CNN
 F 3 "" H 9030 14825 50  0001 C CNN
 	1    9030 14825
@@
 F 0 "C30" V 6295 7575 50  0000 L CNN
 F 1 ".1u" V 6145 7325 50  0000 L CNN
-F 2 "Capacitors_SMD:C_0603" H 6258 7350 50  0001 C CNN
+F 2 "Capacitors_SMD:C_0402" H 6258 7350 50  0001 C CNN
 F 3 "" H 6220 7500 50  0001 C CNN
 	1    6220 7500

Commit message: placed major coponents, no routing
Parts:
- TP3: value 5V0_PWR -> 5V0_MCU
- TP4: value 3V3_PWR -> 3V3_MCU
Connections:
- net GNDPWR: no longer D8.1 (A1)
- net at F1.2, J4.1: now also D8.1 (A1)
Changed lines of the file:
@@
 U 1 1 5C7225B3
 P 16550 8845
-F 0 "U14" H 16350 9270 50  0000 R CNN
+F 0 "U14" H 16945 8485 50  0000 R CNN
 F 1 "ACPL-C87A" H 16210 9115 50  0000 R CNN
 F 2 "Housings_SOIC:SSO-8_6.8x5.9mm_Pitch1.27mm_Clearance8mm" H 16700 8495 50  0001 L CIN
@@
 	0    1    1    0
 $EndComp
-Wire Wire Line
-	2330 7065 2330 6900
-Connection ~ 2330 6900
 $Comp
 L GNDPWR #PWR080
@@
 P 15975 3275
 F 0 "TP3" H 15975 3575 50  0000 C BNN
-F 1 "5V0_PWR" H 15975 3525 50  0000 C CNN
+F 1 "5V0_MCU" H 15975 3525 50  0000 C CNN
 F 2 "Measurement_Points:Measurement_Point_Square-SMD-Pad_Small" H 15975 3275 50  0001 C CNN
 F 3 "" H 15975 3275 50  0001 C CNN
@@
 P 19190 3285
 F 0 "TP4" H 19190 3585 50  0000 C BNN
-F 1 "3V3_PWR" H 19190 3535 50  0000 C CNN
+F 1 "3V3_MCU" H 19190 3535 50  0000 C CNN
 F 2 "Measurement_Points:Measurement_Point_Square-SMD-Pad_Small" H 19190 3285 50  0001 C CNN
 F 3 "" H 19190 3285 50  0001 C CNN
@@
 	1    0    0    -1
 $EndComp
+Connection ~ 2330 6700
+Wire Wire Line
+	2330 7065 2330 6700
+Wire Wire Line
+	2330 6700 2335 6700
 $EndSCHEMATC
