File: nRF24L01_mtr_driver/nRF24L01_mtr_driver.sch (KiCad schematic (older format))
At the start: 133 parts, among them J1 Micro USB, J2 I/O, J4 VBAT, J5 MTR, J6 SERVO, J7 ICSP, Q1 AO4484, Q2 AO4484, Q3 AO4484, Q4 AO4484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

Commit message: Added BOM, changed Vin_min to 6V on silkscreen
Parts:
- U3: value AMS1117-3.3 -> AZ1117EH-3.3TRG1
Other:
- note added: "5.75V-18V"
- note removed: "4.75V-18V"
Changed lines of the file:
@@
 P 9885 4890
 F 0 "U3" H 9484 5110 50  0000 L BNN
-F 1 "AMS1117-3.3" H 9484 4570 50  0000 L BNN
+F 1 "AZ1117EH-3.3TRG1" H 9484 4570 50  0000 L BNN
 F 2 "AMS1117-3.3:SOT229P700X180-4N" H 9885 4890 50  0001 L BNN
 F 3 "Unavailable" H 9885 4890 50  0001 L BNN
@@
 3V3_MCU
 Text Notes 25885 7365 1    118  ~ 0
-4.75V-18V
+5.75V-18V
 Text Notes 17890 7895 1    118  ~ 0
 5V, 2A
